Commit message: Added inertia & collision tag

File: src/my_robot_description/urdf/common_properties.xacro (robot description, xacro)
@@ -10,3 +10,14 @@
         <color rgba ="0 0 1 1" />
     </material>
+<xacro:macro name="box_inertia" params="m x y z o_xyz o_rpy">
+    <inertial>
+        <origin xyz="${o_xyz}" rpy="${o_rpy}"/>
+        <mass value="${m}"/>
+        <inertia
+            ixx="${(m/12) * (y*y + z*z)}"
+            iyy="${(m/12) * (x*x + z*z)}"
+            izz="${(m/12) * (x*x + y*y)}"
+            ixy="0" ixz="0" iyz="0"/>
+    </inertial>
+</xacro:macro>
 </robot>

File: src/my_robot_description/urdf/mobile_base.xacro (robot description, xacro)
@@ -4,5 +4,5 @@
     <xacro:property name="wheel_width"  value="0.05"/>
     <xacro:property name="base_length"  value="0.6"/>
-    <xacro:property name="base_width"  value="0.4"/>\
+    <xacro:property name="base_width"  value="0.4"/>
     <xacro:property name="base_height"  value="0.2"/>
     <link name= "base_footprint_link">
@@ -19,4 +19,13 @@
             <material name= "blue" />
         </visual>
+        <collision>
+            <geometry>
+                <box size = "${base_length} ${base_width} ${base_height}" /> <!-- all dimensions are in meters -->
+            </geometry>
+            <origin xyz = "0 0 0.1" rpy = "0 0 0"/>
+        </collision>
+        <xacro:box_inertia m="5.0" x="${base_length}" y="${base_width}" z="${base_height}"
+                            o_xyz="0 0 ${base_height / 2}" o_rpy="0 0 0"
+        />
     </link>
     <link name= "imu_link">
@@ -28,4 +37,12 @@
             <material name= "green" />
         </visual>
+        <collision>
+            <geometry>
+                <box size = "0.2 0.1 0.05" />
+            </geometry>
+            <origin xyz = "0 0 0.025" rpy = "0 0 0"/>
+        </collision>
+        <xacro:box_inertia m="0.2" x="${base_height}" y="${base_height / 2}" z="0.05"
+                            o_xyz="0 0 0.025" o_rpy="0 0 0" />
     </link>
     <xacro:macro name="wheel_link" params="prefix name" >
@@ -38,4 +55,19 @@
                 <material name= "black" />
             </visual>
+            <collision>
+                <geometry>
+                    <sphere radius = "${wheel_radius}"/>
+                </geometry>
+                <origin xyz = "0 0 0" rpy = "${pi / 2} 0 0"/>
+            </collision>
+            <inertial>
+                <origin xyz="0 0 0" rpy="0 0 0"/>
+                <mass value="0.5"/>
+                <inertia
+                    ixx="${0.5 * 0.5 * wheel_radius * wheel_radius}"
+                    iyy="${(1/12) * 0.5 * (3 * wheel_radius * wheel_radius + wheel_width * wheel_width)}"
+                    izz="${(1/12) * 0.5 * (3 * wheel_radius * wheel_radius + wheel_width * wheel_width)}"
+                    ixy="0" ixz="0" iyz="0"/>
+            </inertial>
         </link>
     </xacro:macro>
@@ -50,4 +82,19 @@
             <material name= "black" />
         </visual>
+        <collision>
+            <geometry>
+                <sphere radius = "0.05"/>
+            </geometry>
+            <origin xyz = "0 0 -0.025" rpy = "${pi / 2} 0 0"/>
+        </collision>
+        <inertial>
+            <origin xyz="0 0 0" rpy="0 0 0"/>
+            <mass value="0.2"/>
+            <inertia
+                ixx="${(2/5) * 0.2 * 0.05 * 0.05}"
+                iyy="${(2/5) * 0.2 * 0.05 * 0.05}"
+                izz="${(2/5) * 0.2 * 0.05 * 0.05}"
+                ixy="0" ixz="0" iyz="0"/>
+        </inertial>
     </link>
     <joint name = "base_footprint_joint" type="fixed" >
