Commit message: Add mobile base URDF, Gazebo xacro, bringup and RViz config

File: src/my_robot_description/urdf/mobile_base.xacro (robot description, xacro)
@@ -7,7 +7,7 @@
     <xacro:property name="base_height"  value="0.2"/>
     <link name= "base_footprint_link">
-        <visual>
+        <!-- <visual>
             <origin xyz = "0 0 0" rpy = "0 0 0"/>
-        </visual>
+        </visual> -->
     </link>
     <link name= "base_link">

File: src/my_robot_description/urdf/my_robot.urdf.xacro (robot description, xacro)
@@ -3,3 +3,4 @@
     <xacro:include filename="$(find my_robot_description)/urdf/common_properties.xacro"/>
     <xacro:include filename="$(find my_robot_description)/urdf/mobile_base.xacro"/>
+    <xacro:include filename="$(find my_robot_description)/urdf/mobile_base_gazebo.xacro"/>
 </robot>

Commit message: added lidar link

File: src/my_robot_description/urdf/mobile_base.xacro (robot description, xacro)
@@ -3,7 +3,8 @@
     <xacro:property name="wheel_radius" value="0.1"/>
     <xacro:property name="wheel_width"  value="0.05"/>
-    <xacro:property name="base_length"  value="0.6"/>
+    <xacro:property name="base_length"  value="0.8"/>
     <xacro:property name="base_width"  value="0.4"/>
     <xacro:property name="base_height"  value="0.2"/>
+    <xacro:property name="lidar" value="0.05" />
     <link name= "base_footprint_link">
         <!-- <visual>
@@ -72,4 +73,27 @@
         </link>
     </xacro:macro>
+    <link name ="lidar_link" >
+        <visual>
+            <geometry>
+                <cylinder radius="${lidar}" length="${lidar}"/>
+            </geometry>
+            <origin xyz="0 0 0.025" rpy="0 0 0" />
+        </visual>
+        <collision>
+            <geometry>
+                <cylinder radius="${lidar}" length="${lidar}"/>
+            </geometry>
+            <origin xyz="0 0 0.025" rpy="0 0 0" />
+        </collision>
+            <inertial>
+                <origin xyz="0 0 0.025" rpy="0 0 0"/>
+                <mass value="0.5"/>
+                <inertia
+                    ixx="${0.5 * 0.5 * lidar * lidar}"
+                    iyy="${(1/12) * 0.5 * (3 * lidar * lidar + lidar * lidar)}"
+                    izz="${(1/12) * 0.5 * (3 * lidar * lidar + lidar * lidar)}"
+                    ixy="0" ixz="0" iyz="0"/>
+            </inertial>
+    </link>
     <xacro:wheel_link prefix="left_"  name="wheel_link"/>
     <xacro:wheel_link prefix="right_" name="wheel_link"/>
@@ -106,5 +130,5 @@
         <parent link="base_link" />
         <child link="imu_link" />
-        <origin xyz="0 0 ${base_height}" rpy="0 0 0"/>
+        <origin xyz="-0.2 0 ${base_height}" rpy="0 0 ${pi /2}"/>
     </joint>
     <joint name="base_left_wheel_joint" type="continuous">
@@ -125,3 +149,9 @@
         <origin xyz="${base_height} 0 -0.025" rpy="0 0 0"/>
     </joint>
+    <joint name="base_lidar_joint" type="continuous">
+        <parent link="base_link" />
+        <child link="lidar_link" />
+        <origin xyz="0.2 0 ${base_height}" rpy="0 0 0"/>
+        <axis xyz="0 0 1" />
+    </joint>
 </robot>
